File: heishamon-lr-pdc.kicad_pcb (KiCad board)
At the start: 2 copper layers, 49.2 x 66.5 mm, 30 parts, among them CN1 S05B-XASK-1(LF)(SN), CN2 S05B-XASK-1(LF)(SN), J1 Conn_01x04_Pin, J2 ESP_SER_DBG, J3 VCC_IN, U1 ISO7762FDW, U2 B1203S-2WR2_C19272681, U3 ESP32-C3-DevKitC-02

Commit message: Update
Parts:
- C2, C4, C5: value CL21A475KAQNNNE -> 10 uF
- U1: value ISO7762FDW -> IS3862LW or ISO7762FDW
- U2: value B1203S-2WR2_C19272681 -> B1205S-2WR2_C2992386
- moved C5 0.10 mm to (50.8, 61.4)
Connections:
- net +12_PDC renamed +12_HP
- net +5_PDC renamed +5_HP
- net /RX (PDC <) renamed /RX (HP <)
- net /TX (PDC >) renamed /TX (HP >)
Routing:
- net +5V: track 8.27 -> 15.6 mm
- net Net-(CN1-Pad3): track 2.17 -> 7.25 mm
- net Net-(CN1-Pad2): track 5.94 -> 10.2 mm
- net +5_HP: track 55.2 -> 55.8 mm
- net /RX (HP <): track 37.4 -> 38.0 mm
Other:
- board text added: "Aquarea HeishaMon Module by LR"
- board text removed: "Aquarea HA Module by LR"
